Commit message: rm: physics in urdf 2.0

File: hexapod_ws/src/hexapod_description/urdf/body.urdf.xacro (robot description, xacro)
@@ -19,7 +19,5 @@
       </collision>
       <inertial>
-        <mass value="0.5"/>
         <origin xyz="0 0 0" rpy="0 0 0"/>
-        <inertia ixx="0.002" ixy="0.0" ixz="0.0" iyy="0.002" iyz="0.0" izz="0.003"/>
       </inertial>
     </link>
@@ -41,7 +39,5 @@
       </collision>
       <inertial>
-        <mass value="0.05"/>
         <origin xyz="0 0 0" rpy="0 0 0"/>
-        <inertia ixx="0.0001" ixy="0.0" ixz="0.0" iyy="0.0001" iyz="0.0" izz="0.0001"/>
       </inertial>
     </link>
@@ -68,7 +64,5 @@
       </collision>
       <inertial>
-        <mass value="0.05"/>
         <origin xyz="0 0 0" rpy="0 0 0"/>
-        <inertia ixx="0.0001" ixy="0.0" ixz="0.0" iyy="0.0001" iyz="0.0" izz="0.0001"/>
       </inertial>
     </link>

Commit message: add: idfk, gazebo sim ig

File: hexapod_ws/src/hexapod_description/urdf/body.urdf.xacro (robot description, xacro)
@@ -20,4 +20,9 @@
       <inertial>
         <origin xyz="0 0 0" rpy="0 0 0"/>
+        <mass value="3.0"/>
+        <inertia
+          ixx="0.5" ixy="0.0" ixz="0.0"
+          iyy="0.5" iyz="0.0"
+          izz="0.5"/>
       </inertial>
     </link>
@@ -40,4 +45,9 @@
       <inertial>
         <origin xyz="0 0 0" rpy="0 0 0"/>
+        <mass value="0.2"/>
+        <inertia
+          ixx="0.005" ixy="0.0" ixz="0.0"
+          iyy="0.005" iyz="0.0"
+          izz="0.005"/>
       </inertial>
     </link>
@@ -65,4 +75,9 @@
       <inertial>
         <origin xyz="0 0 0" rpy="0 0 0"/>
+        <mass value="0.2"/>
+        <inertia
+          ixx="0.005" ixy="0.0" ixz="0.0"
+          iyy="0.005" iyz="0.0"
+          izz="0.005"/>
       </inertial>
     </link>

File: hexapod_ws/src/hexapod_description/urdf/hexapod.urdf.xacro (robot description, xacro)
@@ -10,3 +10,107 @@
   <xacro:hexapod_leg side="right" prefix="r2" x_pos="0.8" y_pos="0" z_pos="0.0" yaw_rot="0"/>
   <xacro:hexapod_leg side="right" prefix="r3" x_pos="0.6" y_pos="-0.8" z_pos="0.0" yaw_rot="-0.78"/>
+    <!-- ros2_control: interfaces for all 18 movable joints -->
+  <ros2_control name="GazeboSimSystem" type="system">
+    <hardware>
+      <plugin>gz_ros2_control/GazeboSimSystem</plugin>
+    </hardware>
+    <joint name="l1_coxa_joint">
+      <command_interface name="position"/>
+      <state_interface name="position"/>
+      <state_interface name="velocity"/>
+    </joint>
+    <joint name="l1_femur_joint">
+      <command_interface name="position"/>
+      <state_interface name="position"/>
+      <state_interface name="velocity"/>
+    </joint>
+    <joint name="l1_tibia_joint">
+      <command_interface name="position"/>
+      <state_interface name="position"/>
+      <state_interface name="velocity"/>
+    </joint>
+    <joint name="l2_coxa_joint">
+      <command_interface name="position"/>
+      <state_interface name="position"/>
+      <state_interface name="velocity"/>
+    </joint>
+    <joint name="l2_femur_joint">
+      <command_interface name="position"/>
+      <state_interface name="position"/>
+      <state_interface name="velocity"/>
+    </joint>
+    <joint name="l2_tibia_joint">
+      <command_interface name="position"/>
+      <state_interface name="position"/>
+      <state_interface name="velocity"/>
+    </joint>
+    <joint name="l3_coxa_joint">
+      <command_interface name="position"/>
+      <state_interface name="position"/>
+      <state_interface name="velocity"/>
+    </joint>
+    <joint name="l3_femur_joint">
+      <command_interface name="position"/>
+      <state_interface name="position"/>
+      <state_interface name="velocity"/>
+    </joint>
+    <joint name="l3_tibia_joint">
+      <command_interface name="position"/>
+      <state_interface name="position"/>
+      <state_interface name="velocity"/>
+    </joint>
+    <joint name="r1_coxa_joint">
+      <command_interface name="position"/>
+      <state_interface name="position"/>
+      <state_interface name="velocity"/>
+    </joint>
+    <joint name="r1_femur_joint">
+      <command_interface name="position"/>
+      <state_interface name="position"/>
+      <state_interface name="velocity"/>
+    </joint>
+    <joint name="r1_tibia_joint">
+      <command_interface name="position"/>
+      <state_interface name="position"/>
+      <state_interface name="velocity"/>
+    </joint>
+    <joint name="r2_coxa_joint">
+      <command_interface name="position"/>
+      <state_interface name="position"/>
+      <state_interface name="velocity"/>
+    </joint>
+    <joint name="r2_femur_joint">
+      <command_interface name="position"/>
+      <state_interface name="position"/>
+      <state_interface name="velocity"/>
+    </joint>
+    <joint name="r2_tibia_joint">
+      <command_interface name="position"/>
+      <state_interface name="position"/>
+      <state_interface name="velocity"/>
+    </joint>
+    <joint name="r3_coxa_joint">
+      <command_interface name="position"/>
+      <state_interface name="position"/>
+      <state_interface name="velocity"/>
+    </joint>
+    <joint name="r3_femur_joint">
+      <command_interface name="position"/>
+      <state_interface name="position"/>
+      <state_interface name="velocity"/>
+    </joint>
+    <joint name="r3_tibia_joint">
+      <command_interface name="position"/>
+      <state_interface name="position"/>
+      <state_interface name="velocity"/>
+    </joint>
+  </ros2_control>
+  <!-- Gazebo Sim Harmonic integration -->
+  <gazebo>
+    <plugin
+      filename="libgz_ros2_control-system.so"
+      name="gz_ros2_control::GazeboSimROS2ControlPlugin">
+      <parameters>$(find hexapod_description)/config/controllers.yaml</parameters>
+    </plugin>
+  </gazebo>
 </robot>

File: hexapod_ws/src/hexapod_description/urdf/leg.urdf.xacro (robot description, xacro)
@@ -20,4 +20,9 @@
       <inertial>
         <origin xyz="0 0 0" rpy="0 0 0"/>
+        <mass value="0.2"/>
+        <inertia
+          ixx="0.0002" ixy="0.0" ixz="0.0"
+          iyy="0.0028" iyz="0.0"
+          izz="0.0028"/>
       </inertial>
     </link>
@@ -47,4 +52,9 @@
       <inertial>
         <origin xyz="0 0 0" rpy="0 0 0"/>
+        <mass value="0.3"/>
+        <inertia
+          ixx="0.0003" ixy="0.0" ixz="0.0"
+          iyy="0.016" iyz="0.0"
+          izz="0.016"/>
       </inertial>
     </link>
@@ -74,4 +84,9 @@
       <inertial>
         <origin xyz="0 0 0" rpy="0 0 0"/>
+        <mass value="0.2"/>
+        <inertia
+          ixx="0.0001" ixy="0.0" ixz="0.0"
+          iyy="0.011" iyz="0.0"
+          izz="0.011"/>
       </inertial>
     </link>
@@ -101,4 +116,9 @@
       <inertial>
         <origin xyz="0 0 0" rpy="0 0 0"/>
+        <mass value="0.05"/>
+        <inertia
+          ixx="0.0001" ixy="0.0" ixz="0.0"
+          iyy="0.0001" iyz="0.0"
+          izz="0.0001"/>
       </inertial>
     </link>
@@ -126,4 +146,9 @@
       <inertial>
         <origin xyz="0 0 0" rpy="0 0 0"/>
+        <mass value="0.02"/>
+        <inertia
+          ixx="0.00002" ixy="0.0" ixz="0.0"
+          iyy="0.00002" iyz="0.0"
+          izz="0.00002"/>
       </inertial>
     </link>
@@ -151,4 +176,9 @@
       <inertial>
         <origin xyz="0 0 0" rpy="0 0 0"/>
+        <mass value="0.05"/>
+        <inertia
+          ixx="0.0001" ixy="0.0" ixz="0.0"
+          iyy="0.0001" iyz="0.0"
+          izz="0.0001"/>
       </inertial>
     </link>

Commit message: fix: real_time_factor is now higher but not high enough

File: hexapod_ws/src/hexapod_description/urdf/body.urdf.xacro (robot description, xacro)
@@ -14,5 +14,5 @@
       <collision>
         <geometry>
-          <mesh filename="package://hexapod_description/meshes/frame.stl" scale="0.01 0.01 0.01"/>
+          <mesh filename="package://hexapod_description/meshes/frame-collision.stl" scale="0.01 0.01 0.01"/>
         </geometry>
         <origin xyz="0 0 0" rpy="0 0 0"/>
@@ -39,5 +39,5 @@
       <collision>
         <geometry>
-          <mesh filename="package://hexapod_description/meshes/top-cover.stl" scale="0.01 0.01 0.01"/>
+          <mesh filename="package://hexapod_description/meshes/top-cover-collision.stl" scale="0.01 0.01 0.01"/>
         </geometry>
         <origin xyz="0 0 0.125" rpy="0 0 0"/>
@@ -69,5 +69,5 @@
       <collision>
         <geometry>
-          <mesh filename="package://hexapod_description/meshes/bottom-cover.stl" scale="0.01 0.01 0.01"/>
+          <mesh filename="package://hexapod_description/meshes/bottom-cover-collision.stl" scale="0.01 0.01 0.01"/>
         </geometry>
         <origin xyz="0 0 0.2" rpy="0 0 0"/>

File: hexapod_ws/src/hexapod_description/urdf/leg.urdf.xacro (robot description, xacro)
@@ -14,5 +14,5 @@
       <collision>
         <geometry>
-          <mesh filename="package://hexapod_description/meshes/${side}-coxa.stl" scale="0.01 0.01 0.01"/>
+          <mesh filename="package://hexapod_description/meshes/${side}-coxa-collision.stl" scale="0.01 0.01 0.01"/>
         </geometry>
         <origin xyz="0 0 0" rpy="0 0 0"/>
@@ -47,5 +47,5 @@
       <collision>
         <geometry>
-          <mesh filename="package://hexapod_description/meshes/${side}-femur.stl" scale="0.01 0.01 0.01"/>
+          <mesh filename="package://hexapod_description/meshes/${side}-femur-collision.stl" scale="0.01 0.01 0.01"/>
         </geometry>
         <origin xyz="0 ${0.1 if side == 'left' else -0.1} 0" rpy="-1.57 0 0"/>
@@ -80,5 +80,5 @@
       <collision>
         <geometry>
-          <mesh filename="package://hexapod_description/meshes/${side}-tibia.stl" scale="0.01 0.01 0.01"/>
+          <mesh filename="package://hexapod_description/meshes/${side}-tibia-collision.stl" scale="0.01 0.01 0.01"/>
         </geometry>
         <origin xyz="0.5 -0.05 0" rpy="0 0 3.14"/>
@@ -113,5 +113,5 @@
       <collision>
         <geometry>
-          <mesh filename="package://hexapod_description/meshes/shield.stl" scale="0.01 0.01 0.01"/>
+          <mesh filename="package://hexapod_description/meshes/shield-collision.stl" scale="0.01 0.01 0.01"/>
         </geometry>
         <origin xyz="0.4 0.05 0" rpy="0 0 3.14"/>
@@ -143,5 +143,5 @@
       <collision>
         <geometry>
-          <mesh filename="package://hexapod_description/meshes/micro-switch-tip.stl" scale="0.01 0.01 0.01"/>
+          <mesh filename="package://hexapod_description/meshes/micro-switch-tip-collision.stl" scale="0.01 0.01 0.01"/>
         </geometry>
         <origin xyz="0 0 0" rpy="0 0 3.14"/>
@@ -173,5 +173,5 @@
       <collision>
         <geometry>
-          <mesh filename="package://hexapod_description/meshes/tip.stl" scale="0.01 0.01 0.01"/>
+          <mesh filename="package://hexapod_description/meshes/tip-collision.stl" scale="0.01 0.01 0.01"/>
         </geometry>
         <origin xyz="0 0 0" rpy="0 0 0"/>

Commit message: fix: no more collision, just simplest shapes

File: hexapod_ws/src/hexapod_description/urdf/body.urdf.xacro (robot description, xacro)
@@ -5,5 +5,6 @@
       <visual>
         <geometry>
-          <mesh filename="package://hexapod_description/meshes/frame.stl" scale="0.01 0.01 0.01"/>
+          <mesh filename="package://hexapod_description/meshes/frame.stl"
+                scale="0.001 0.001 0.001"/>
         </geometry>
         <origin xyz="0 0 0" rpy="0 0 0"/>
@@ -14,5 +15,5 @@
       <collision>
         <geometry>
-          <mesh filename="package://hexapod_description/meshes/frame-collision.stl" scale="0.01 0.01 0.01"/>
+          <box size="0.198 0.205 0.016"/>
         </geometry>
         <origin xyz="0 0 0" rpy="0 0 0"/>
@@ -22,7 +23,7 @@
         <mass value="3.0"/>
         <inertia
-          ixx="0.5" ixy="0.0" ixz="0.0"
-          iyy="0.5" iyz="0.0"
-          izz="0.5"/>
+          ixx="0.005" ixy="0.0" ixz="0.0"
+          iyy="0.005" iyz="0.0"
+          izz="0.005"/>
       </inertial>
     </link>
@@ -30,24 +31,19 @@
       <visual>
         <geometry>
-          <mesh filename="package://hexapod_description/meshes/top-cover.stl" scale="0.01 0.01 0.01"/>
+          <mesh filename="package://hexapod_description/meshes/top-cover.stl"
+                scale="0.001 0.001 0.001"/>
         </geometry>
-        <origin xyz="0 0 0.125" rpy="0 0 0"/>
+        <origin xyz="0 0 0.0125" rpy="0 0 0"/>
         <material name="orange">
           <color rgba="1.0 0.5 0.0 1.0"/>
         </material>
       </visual>
-      <collision>
-        <geometry>
-          <mesh filename="package://hexapod_description/meshes/top-cover-collision.stl" scale="0.01 0.01 0.01"/>
-        </geometry>
-        <origin xyz="0 0 0.125" rpy="0 0 0"/>
-      </collision>
       <inertial>
         <origin xyz="0 0 0" rpy="0 0 0"/>
         <mass value="0.2"/>
         <inertia
-          ixx="0.005" ixy="0.0" ixz="0.0"
-          iyy="0.005" iyz="0.0"
-          izz="0.005"/>
+          ixx="0.00005" ixy="0.0" ixz="0.0"
+          iyy="0.00005" iyz="0.0"
+          izz="0.00005"/>
       </inertial>
     </link>
@@ -55,29 +51,24 @@
       <parent link="base_link"/>
       <child link="top_cover_link"/>
-      <origin xyz="0 0 0.03" rpy="0 0 0"/>
+      <origin xyz="0 0 0.003" rpy="0 0 0"/>
     </joint>
     <link name="bottom_cover_link">
       <visual>
         <geometry>
-          <mesh filename="package://hexapod_description/meshes/bottom-cover.stl" scale="0.01 0.01 0.01"/>
+          <mesh filename="package://hexapod_description/meshes/bottom-cover.stl"
+                scale="0.001 0.001 0.001"/>
         </geometry>
-        <origin xyz="0 0 0.2" rpy="0 0 0"/>
+        <origin xyz="0 0 0.02" rpy="0 0 0"/>
         <material name="orange">
           <color rgba="1.0 0.5 0.0 1.0"/>
         </material>
       </visual>
-      <collision>
-        <geometry>
-          <mesh filename="package://hexapod_description/meshes/bottom-cover-collision.stl" scale="0.01 0.01 0.01"/>
-        </geometry>
-        <origin xyz="0 0 0.2" rpy="0 0 0"/>
-      </collision>
       <inertial>
         <origin xyz="0 0 0" rpy="0 0 0"/>
         <mass value="0.2"/>
         <inertia
-          ixx="0.005" ixy="0.0" ixz="0.0"
-          iyy="0.005" iyz="0.0"
-          izz="0.005"/>
+          ixx="0.00005" ixy="0.0" ixz="0.0"
+          iyy="0.00005" iyz="0.0"
+          izz="0.00005"/>
       </inertial>
     </link>
@@ -85,5 +76,5 @@
       <parent link="base_link"/>
       <child link="bottom_cover_link"/>
-      <origin xyz="0 0 -0.03" rpy="0 0 0"/>
+      <origin xyz="0 0 -0.003" rpy="0 0 0"/>
     </joint>
   </xacro:macro>

File: hexapod_ws/src/hexapod_description/urdf/hexapod.urdf.xacro (robot description, xacro)
@@ -4,11 +4,19 @@
   <xacro:include filename="$(find hexapod_description)/urdf/leg.urdf.xacro"/>
   <xacro:hexapod_body/>
-  <xacro:hexapod_leg side="left" prefix="l1" x_pos="-0.6" y_pos="0.8" z_pos="0.0" yaw_rot="2.35"/>
-  <xacro:hexapod_leg side="left" prefix="l2" x_pos="-0.8" y_pos="0" z_pos="0.0" yaw_rot="3.14"/>
-  <xacro:hexapod_leg side="left" prefix="l3" x_pos="-0.6" y_pos="-0.8" z_pos="0.0" yaw_rot="-2.35"/>
-  <xacro:hexapod_leg side="right" prefix="r1" x_pos="0.6" y_pos="0.8" z_pos="0.0" yaw_rot="0.78"/>
-  <xacro:hexapod_leg side="right" prefix="r2" x_pos="0.8" y_pos="0" z_pos="0.0" yaw_rot="0"/>
-  <xacro:hexapod_leg side="right" prefix="r3" x_pos="0.6" y_pos="-0.8" z_pos="0.0" yaw_rot="-0.78"/>
-    <!-- ros2_control: interfaces for all 18 movable joints -->
+  <!-- Left side -->
+  <xacro:hexapod_leg side="left" prefix="l1"
+                     x_pos="-0.06" y_pos="0.08" z_pos="0.0" yaw_rot="2.35"/>
+  <xacro:hexapod_leg side="left" prefix="l2"
+                     x_pos="-0.08" y_pos="0.0" z_pos="0.0" yaw_rot="3.14"/>
+  <xacro:hexapod_leg side="left" prefix="l3"
+                     x_pos="-0.06" y_pos="-0.08" z_pos="0.0" yaw_rot="-2.35"/>
+  <!-- Right side -->
+  <xacro:hexapod_leg side="right" prefix="r1"
+                     x_pos="0.06" y_pos="0.08" z_pos="0.0" yaw_rot="0.78"/>
+  <xacro:hexapod_leg side="right" prefix="r2"
+                     x_pos="0.08" y_pos="0.0" z_pos="0.0" yaw_rot="0"/>
+  <xacro:hexapod_leg side="right" prefix="r3"
+                     x_pos="0.06" y_pos="-0.08" z_pos="0.0" yaw_rot="-0.78"/>
+  <!-- ros2_control: interfaces for all 18 movable joints -->
   <ros2_control name="GazeboSimSystem" type="system">
     <hardware>

File: hexapod_ws/src/hexapod_description/urdf/leg.urdf.xacro (robot description, xacro)
@@ -5,5 +5,6 @@
       <visual>
         <geometry>
-          <mesh filename="package://hexapod_description/meshes/${side}-coxa.stl" scale="0.01 0.01 0.01"/>
+          <mesh filename="package://hexapod_description/meshes/${side}-coxa.stl"
+                scale="0.001 0.001 0.001"/>
         </geometry>
         <origin xyz="0 0 0" rpy="0 0 0"/>
@@ -12,10 +13,4 @@
         </material>
       </visual>
-      <collision>
-        <geometry>
-          <mesh filename="package://hexapod_description/meshes/${side}-coxa-collision.stl" scale="0.01 0.01 0.01"/>
-        </geometry>
-        <origin xyz="0 0 0" rpy="0 0 0"/>
-      </collision>
       <inertial>
         <origin xyz="0 0 0" rpy="0 0 0"/>
@@ -38,17 +33,13 @@
       <visual>
         <geometry>
-          <mesh filename="package://hexapod_description/meshes/${side}-femur.stl" scale="0.01 0.01 0.01"/>
+          <mesh filename="package://hexapod_description/meshes/${side}-femur.stl"
+                scale="0.001 0.001 0.001"/>
         </geometry>
-        <origin xyz="0 ${0.1 if side == 'left' else -0.1} 0" rpy="-1.57 0 0"/>
+        <origin xyz="0 ${0.01 if side == 'left' else -0.01} 0"
+                rpy="-1.57 0 0"/>
         <material name="orange">
           <color rgba="1.0 0.5 0.0 1.0"/>
         </material>
       </visual>
-      <collision>
-        <geometry>
-          <mesh filename="package://hexapod_description/meshes/${side}-femur-collision.stl" scale="0.01 0.01 0.01"/>
-        </geometry>
-        <origin xyz="0 ${0.1 if side == 'left' else -0.1} 0" rpy="-1.57 0 0"/>
-      </collision>
       <inertial>
         <origin xyz="0 0 0" rpy="0 0 0"/>
@@ -63,5 +54,5 @@
       <parent link="${prefix}_coxa_link"/>
       <child link="${prefix}_femur_link"/>
-      <origin xyz="0.4 0 0.05" rpy="0 -0.78 0"/>
+      <origin xyz="0.04 0 0.005" rpy="0 -0.78 0"/>
       <axis xyz="0 1 0"/>
       <limit lower="-1.57" upper="1.57" effort="100.0" velocity="3.0"/>
@@ -71,17 +62,12 @@
       <visual>
         <geometry>
-          <mesh filename="package://hexapod_description/meshes/${side}-tibia.stl" scale="0.01 0.01 0.01"/>
+          <mesh filename="package://hexapod_description/meshes/${side}-tibia.stl"
+                scale="0.001 0.001 0.001"/>
         </geometry>
-        <origin xyz="0.5 -0.05 0" rpy="0 0 3.14"/>
+        <origin xyz="0.05 -0.005 0" rpy="0 0 3.14"/>
         <material name="orange">
           <color rgba="1.0 0.5 0.0 1.0"/>
         </material>
       </visual>
-      <collision>
-        <geometry>
-          <mesh filename="package://hexapod_description/meshes/${side}-tibia-collision.stl" scale="0.01 0.01 0.01"/>
-        </geometry>
-        <origin xyz="0.5 -0.05 0" rpy="0 0 3.14"/>
-      </collision>
       <inertial>
         <origin xyz="0 0 0" rpy="0 0 0"/>
@@ -96,5 +82,5 @@
       <parent link="${prefix}_femur_link"/>
       <child link="${prefix}_tibia_link"/>
-      <origin xyz="0.8 0 0" rpy="0 0.78 0"/>
+      <origin xyz="0.08 0 0" rpy="0 0.078 0"/>
       <axis xyz="0 1 0"/>
       <limit lower="-1.57" upper="1.57" effort="100.0" velocity="3.0"/>
@@ -104,17 +90,12 @@
       <visual>
         <geometry>
-          <mesh filename="package://hexapod_description/meshes/shield.stl" scale="0.01 0.01 0.01"/>
+          <mesh filename="package://hexapod_description/meshes/shield.stl"
+                scale="0.001 0.001 0.001"/>
         </geometry>
-        <origin xyz="0.4 0.05 0" rpy="0 0 3.14"/>
+        <origin xyz="0.04 0.005 0" rpy="0 0 3.14"/>
         <material name="orange">
           <color rgba="1.0 0.5 0.0 1.0"/>
         </material>
       </visual>
-      <collision>
-        <geometry>
-          <mesh filename="package://hexapod_description/meshes/shield-collision.stl" scale="0.01 0.01 0.01"/>
-        </geometry>
-        <origin xyz="0.4 0.05 0" rpy="0 0 3.14"/>
-      </collision>
       <inertial>
         <origin xyz="0 0 0" rpy="0 0 0"/>
@@ -129,10 +110,11 @@
       <parent link="${prefix}_tibia_link"/>
       <child link="${prefix}_shield_link"/>
-      <origin xyz="0.1 0 0" rpy="0 0 0"/>
+      <origin xyz="0.01 0 0" rpy="0 0 0"/>
     </joint>
     <link name="${prefix}_micro_switch_tip_link">
       <visual>
         <geometry>
-          <mesh filename="package://hexapod_description/meshes/micro-switch-tip.stl" scale="0.01 0.01 0.01"/>
+          <mesh filename="package://hexapod_description/meshes/micro-switch-tip.stl"
+                scale="0.001 0.001 0.001"/>
         </geometry>
         <origin xyz="0 0 0" rpy="0 0 3.14"/>
@@ -141,10 +123,4 @@
         </material>
       </visual>
-      <collision>
-        <geometry>
-          <mesh filename="package://hexapod_description/meshes/micro-switch-tip-collision.stl" scale="0.01 0.01 0.01"/>
-        </geometry>
-        <origin xyz="0 0 0" rpy="0 0 3.14"/>
-      </collision>
       <inertial>
         <origin xyz="0 0 0" rpy="0 0 0"/>
@@ -159,10 +135,11 @@
       <parent link="${prefix}_tibia_link"/>
       <child link="${prefix}_micro_switch_tip_link"/>
-      <origin xyz="0.4 0 -1.3" rpy="0 0 0"/>
+      <origin xyz="0.04 0 -0.13" rpy="0 0 0"/>
     </joint>
     <link name="${prefix}_tip_link">
       <visual>
         <geometry>
-          <mesh filename="package://hexapod_description/meshes/tip.stl" scale="0.01 0.01 0.01"/>
+          <mesh filename="package://hexapod_description/meshes/tip.stl"
+                scale="0.001 0.001 0.001"/>
         </geometry>
         <origin xyz="0 0 0" rpy="0 0 0"/>
@@ -173,5 +150,5 @@
       <collision>
         <geometry>
-          <mesh filename="package://hexapod_description/meshes/tip-collision.stl" scale="0.01 0.01 0.01"/>
+          <sphere radius="0.005"/>
         </geometry>
         <origin xyz="0 0 0" rpy="0 0 0"/>
@@ -191,4 +168,8 @@
       <origin xyz="0 0 0" rpy="0 0 0"/>
     </joint>
+    <gazebo reference="${prefix}_tip_link">
+      <mu1>1.0</mu1>
+      <mu2>1.0</mu2>
+    </gazebo>
   </xacro:macro>
 </robot>
