Commit message: fix: realistic inertial

File: hexapod_ws/src/hexapod_description/urdf/body.urdf.xacro (robot description, xacro)
@@ -20,10 +20,7 @@
       </collision>
       <inertial>
-        <origin xyz="0 0 0" rpy="0 0 0"/>
-        <mass value="3.0"/>
-        <inertia
-          ixx="0.005" ixy="0.0" ixz="0.0"
-          iyy="0.005" iyz="0.0"
-          izz="0.005"/>
+        <origin xyz="-0.00002 -0.00106 0.00800" rpy="0 0 0"/>
+        <mass value="0.4864"/>
+        <inertia ixx="1.763e-03" ixy="-5.177e-08" ixz="5.397e-10" iyy="1.708e-03" iyz="2.214e-09" izz="3.371e-03"/>
       </inertial>
     </link>
@@ -40,10 +37,7 @@
       </visual>
       <inertial>
-        <origin xyz="0 0 0" rpy="0 0 0"/>
-        <mass value="0.2"/>
-        <inertia
-          ixx="0.00005" ixy="0.0" ixz="0.0"
-          iyy="0.00005" iyz="0.0"
-          izz="0.00005"/>
+        <origin xyz="0.00000 -0.00000 0.04655" rpy="0 0 0"/>
+        <mass value="0.1846"/>
+        <inertia ixx="1.510e-04" ixy="1.687e-10" ixz="4.441e-11" iyy="2.034e-04" iyz="-1.877e-10" izz="2.428e-04"/>
       </inertial>
     </link>
@@ -65,10 +59,7 @@
       </visual>
       <inertial>
-        <origin xyz="0 0 0" rpy="0 0 0"/>
-        <mass value="0.2"/>
-        <inertia
-          ixx="0.00005" ixy="0.0" ixz="0.0"
-          iyy="0.00005" iyz="0.0"
-          izz="0.00005"/>
+        <origin xyz="0.00054 0.00110 -0.01698" rpy="0 0 0"/>
+        <mass value="0.4426"/>
+        <inertia ixx="7.003e-04" ixy="-3.336e-06" ixz="-4.496e-06" iyy="1.982e-04" iyz="-2.872e-06" izz="7.458e-04"/>
       </inertial>
     </link>

File: hexapod_ws/src/hexapod_description/urdf/hexapod.urdf.xacro (robot description, xacro)
@@ -4,5 +4,4 @@
   <xacro:include filename="$(find hexapod_description)/urdf/leg.urdf.xacro"/>
   <xacro:hexapod_body/>
-  <!-- Left side -->
   <xacro:hexapod_leg side="left" prefix="l1"
                      x_pos="-0.06" y_pos="0.08" z_pos="0.0" yaw_rot="2.35"/>
@@ -11,5 +10,4 @@
   <xacro:hexapod_leg side="left" prefix="l3"
                      x_pos="-0.06" y_pos="-0.08" z_pos="0.0" yaw_rot="-2.35"/>
-  <!-- Right side -->
   <xacro:hexapod_leg side="right" prefix="r1"
                      x_pos="0.06" y_pos="0.08" z_pos="0.0" yaw_rot="0.78"/>
@@ -18,5 +16,4 @@
   <xacro:hexapod_leg side="right" prefix="r3"
                      x_pos="0.06" y_pos="-0.08" z_pos="0.0" yaw_rot="-0.78"/>
-  <!-- ros2_control: interfaces for all 18 movable joints -->
   <ros2_control name="GazeboSimSystem" type="system">
     <hardware>
@@ -114,5 +111,4 @@
     </joint>
   </ros2_control>
-  <!-- Gazebo Sim Harmonic integration -->
   <gazebo>
     <plugin

File: hexapod_ws/src/hexapod_description/urdf/leg.urdf.xacro (robot description, xacro)
@@ -14,10 +14,7 @@
       </visual>
       <inertial>
-        <origin xyz="0 0 0" rpy="0 0 0"/>
-        <mass value="0.2"/>
-        <inertia
-          ixx="0.0002" ixy="0.0" ixz="0.0"
-          iyy="0.0028" iyz="0.0"
-          izz="0.0028"/>
+        <origin xyz="0.02964 0.00014 0.00625" rpy="0 0 0"/>
+        <mass value="0.0771"/>
+        <inertia ixx="1.617e-05" ixy="4.643e-08" ixz="6.122e-07" iyy="1.852e-05" iyz="-6.164e-08" izz="1.885e-05"/>
       </inertial>
     </link>
@@ -27,5 +24,5 @@
       <origin xyz="${x_pos} ${y_pos} ${z_pos}" rpy="0 0 ${yaw_rot}"/>
       <axis xyz="0 0 1"/>
-      <limit lower="-1.57" upper="1.57" effort="100.0" velocity="3.0"/>
+      <limit lower="-1.57" upper="1.57" effort="3.4" velocity="5.0"/>
       <dynamics damping="0.5" friction="0.05"/>
     </joint>
@@ -43,10 +40,7 @@
       </visual>
       <inertial>
-        <origin xyz="0 0 0" rpy="0 0 0"/>
-        <mass value="0.3"/>
-        <inertia
-          ixx="0.0003" ixy="0.0" ixz="0.0"
-          iyy="0.016" iyz="0.0"
-          izz="0.016"/>
+        <origin xyz="0.06445 -0.00082 -0.00021" rpy="0 0 0"/>
+        <mass value="0.0814"/>
+        <inertia ixx="1.867e-05" ixy="-1.515e-06" ixz="-4.656e-07" iyy="2.912e-05" iyz="-7.096e-08" izz="4.288e-05"/>
       </inertial>
     </link>
@@ -56,5 +50,5 @@
       <origin xyz="0.04 0 0.005" rpy="0 -0.78 0"/>
       <axis xyz="0 1 0"/>
-      <limit lower="-1.57" upper="1.57" effort="100.0" velocity="3.0"/>
+      <limit lower="-1.57" upper="1.57" effort="3.4" velocity="5.0"/>
       <dynamics damping="0.5" friction="0.05"/>
     </joint>
@@ -71,10 +65,7 @@
       </visual>
       <inertial>
-        <origin xyz="0 0 0" rpy="0 0 0"/>
-        <mass value="0.2"/>
-        <inertia
-          ixx="0.0001" ixy="0.0" ixz="0.0"
-          iyy="0.011" iyz="0.0"
-          izz="0.011"/>
+        <origin xyz="0.02796 0.00030 -0.03451" rpy="0 0 0"/>
+        <mass value="0.0112"/>
+        <inertia ixx="1.178e-05" ixy="1.476e-07" ixz="5.850e-06" iyy="1.578e-05" iyz="-2.169e-07" izz="4.209e-06"/>
       </inertial>
     </link>
@@ -84,5 +75,5 @@
       <origin xyz="0.08 0 0" rpy="0 0.078 0"/>
       <axis xyz="0 1 0"/>
-      <limit lower="-1.57" upper="1.57" effort="100.0" velocity="3.0"/>
+      <limit lower="-1.57" upper="1.57" effort="3.4" velocity="5.0"/>
       <dynamics damping="0.5" friction="0.05"/>
     </joint>
@@ -99,10 +90,7 @@
       </visual>
       <inertial>
-        <origin xyz="0 0 0" rpy="0 0 0"/>
-        <mass value="0.05"/>
-        <inertia
-          ixx="0.0001" ixy="0.0" ixz="0.0"
-          iyy="0.0001" iyz="0.0"
-          izz="0.0001"/>
+        <origin xyz="0.02928 0.00052 -0.04358" rpy="0 0 0"/>
+        <mass value="0.0098"/>
+        <inertia ixx="1.094e-05" ixy="-6.245e-10" ixz="2.948e-06" iyy="1.025e-05" iyz="-6.117e-09" izz="3.014e-06"/>
       </inertial>
     </link>
@@ -124,10 +112,7 @@
       </visual>
       <inertial>
-        <origin xyz="0 0 0" rpy="0 0 0"/>
-        <mass value="0.02"/>
-        <inertia
-          ixx="0.00002" ixy="0.0" ixz="0.0"
-          iyy="0.00002" iyz="0.0"
-          izz="0.00002"/>
+        <origin xyz="0.00621 -0.00001 0.02072" rpy="0 0 0"/>
+        <mass value="0.0041"/>
+        <inertia ixx="1.977e-07" ixy="2.657e-11" ixz="-4.968e-08" iyy="2.338e-07" iyz="5.395e-11" izz="1.167e-07"/>
       </inertial>
     </link>
@@ -155,10 +140,7 @@
       </collision>
       <inertial>
-        <origin xyz="0 0 0" rpy="0 0 0"/>
-        <mass value="0.05"/>
-        <inertia
-          ixx="0.0001" ixy="0.0" ixz="0.0"
-          iyy="0.0001" iyz="0.0"
-          izz="0.0001"/>
+        <origin xyz="0.00000 -0.00000 -0.00309" rpy="0 0 0"/>
+        <mass value="0.0018"/>
+        <inertia ixx="1.069e-08" ixy="6.542e-14" ixz="-2.181e-12" iyy="1.069e-08" iyz="3.638e-12" izz="2.687e-09"/>
       </inertial>
     </link>
