Commit message: add: base urdf and rviz2 visualization

File: hexapod_ws/src/hexapod_description/urdf/leg.urdf.xacro (robot description, xacro)
@@ -1,10 +1,11 @@
 <?xml version="1.0"?>
 <robot xmlns:xacro="http://www.ros.org/wiki/xacro">
-  <xacro:macro name="hexapod_leg" params="side prefix x_pos y_pos yaw_rot">
+  <xacro:macro name="hexapod_leg" params="side prefix x_pos y_pos z_pos yaw_rot">
     <link name="${prefix}_coxa_link">
       <visual>
         <geometry>
-          <mesh filename="package://hexapod_description/meshes/${side}-coxa.stl" scale="0.001 0.001 0.001"/>
+          <mesh filename="package://hexapod_description/meshes/${side}-coxa.stl" scale="0.01 0.01 0.01"/>
         </geometry>
+        <origin xyz="0 0 0" rpy="0 0 0"/>
         <material name="orange">
           <color rgba="1.0 0.5 0.0 1.0"/>
@@ -13,6 +14,7 @@
       <collision>
         <geometry>
-          <mesh filename="package://hexapod_description/meshes/${side}-coxa.stl" scale="0.001 0.001 0.001"/>
+          <mesh filename="package://hexapod_description/meshes/${side}-coxa.stl" scale="0.01 0.01 0.01"/>
         </geometry>
+        <origin xyz="0 0 0" rpy="0 0 0"/>
       </collision>
       <inertial>
@@ -25,5 +27,5 @@
       <parent link="base_link"/>
       <child link="${prefix}_coxa_link"/>
-      <origin xyz="${x_pos} ${y_pos} 0" rpy="0 0 ${yaw_rot}"/>
+      <origin xyz="${x_pos} ${y_pos} ${z_pos}" rpy="0 0 ${yaw_rot}"/>
       <axis xyz="0 0 1"/>
       <limit lower="-1.57" upper="1.57" effort="2.0" velocity="1.0"/>
@@ -32,6 +34,7 @@
       <visual>
         <geometry>
-          <mesh filename="package://hexapod_description/meshes/${side}-femur.stl" scale="0.001 0.001 0.001"/>
+          <mesh filename="package://hexapod_description/meshes/${side}-femur.stl" scale="0.01 0.01 0.01"/>
         </geometry>
+        <origin xyz="0 ${0.1 if side == 'left' else -0.1} 0" rpy="-1.57 0 0"/>
         <material name="orange">
           <color rgba="1.0 0.5 0.0 1.0"/>
@@ -40,6 +43,7 @@
       <collision>
         <geometry>
-          <mesh filename="package://hexapod_description/meshes/${side}-femur.stl" scale="0.001 0.001 0.001"/>
+          <mesh filename="package://hexapod_description/meshes/${side}-femur.stl" scale="0.01 0.01 0.01"/>
         </geometry>
+        <origin xyz="0 ${0.1 if side == 'left' else -0.1} 0" rpy="-1.57 0 0"/>
       </collision>
       <inertial>
@@ -52,5 +56,5 @@
       <parent link="${prefix}_coxa_link"/>
       <child link="${prefix}_femur_link"/>
-      <origin xyz="0.05 0 0" rpy="0 0 0"/>
+      <origin xyz="0.4 0 0.05" rpy="0 -0.78 0"/>
       <axis xyz="0 1 0"/>
       <limit lower="-1.57" upper="1.57" effort="2.0" velocity="1.0"/>
@@ -59,6 +63,7 @@
       <visual>
         <geometry>
-          <mesh filename="package://hexapod_description/meshes/${side}-tibia.stl" scale="0.001 0.001 0.001"/>
+          <mesh filename="package://hexapod_description/meshes/${side}-tibia.stl" scale="0.01 0.01 0.01"/>
         </geometry>
+        <origin xyz="0.5 -0.05 0" rpy="0 0 3.14"/>
         <material name="orange">
           <color rgba="1.0 0.5 0.0 1.0"/>
@@ -67,6 +72,7 @@
       <collision>
         <geometry>
-          <mesh filename="package://hexapod_description/meshes/${side}-tibia.stl" scale="0.001 0.001 0.001"/>
+          <mesh filename="package://hexapod_description/meshes/${side}-tibia.stl" scale="0.01 0.01 0.01"/>
         </geometry>
+        <origin xyz="0.5 -0.05 0" rpy="0 0 3.14"/>
       </collision>
       <inertial>
@@ -79,8 +85,89 @@
       <parent link="${prefix}_femur_link"/>
       <child link="${prefix}_tibia_link"/>
-      <origin xyz="0.1 0 0" rpy="0 0 0"/>
+      <origin xyz="0.8 0 0" rpy="0 0.78 0"/>
       <axis xyz="0 1 0"/>
       <limit lower="-1.57" upper="1.57" effort="2.0" velocity="1.0"/>
     </joint>
+    <link name="${prefix}_shield_link">
+      <visual>
+        <geometry>
+          <mesh filename="package://hexapod_description/meshes/shield.stl" scale="0.01 0.01 0.01"/>
+        </geometry>
+        <origin xyz="0.4 0.05 0" rpy="0 0 3.14"/>
+        <material name="orange">
+          <color rgba="1.0 0.5 0.0 1.0"/>
+        </material>
+      </visual>
+      <collision>
+        <geometry>
+          <mesh filename="package://hexapod_description/meshes/shield.stl" scale="0.01 0.01 0.01"/>
+        </geometry>
+        <origin xyz="0.4 0.05 0" rpy="0 0 3.14"/>
+      </collision>
+      <inertial>
+        <mass value="0.01"/>
+        <origin xyz="0 0 0" rpy="0 0 0"/>
+        <inertia ixx="0.00001" ixy="0.0" ixz="0.0" iyy="0.00001" iyz="0.0" izz="0.00001"/>
+      </inertial>
+    </link>
+    <joint name="${prefix}_shield_joint" type="fixed">
+      <parent link="${prefix}_tibia_link"/>
+      <child link="${prefix}_shield_link"/>
+      <origin xyz="0.1 0 0" rpy="0 0 0"/>
+    </joint>
+    <link name="${prefix}_micro_switch_tip_link">
+      <visual>
+        <geometry>
+          <mesh filename="package://hexapod_description/meshes/micro-switch-tip.stl" scale="0.01 0.01 0.01"/>
+        </geometry>
+        <origin xyz="0 0 0" rpy="0 0 3.14"/>
+        <material name="orange">
+          <color rgba="1.0 0.5 0.0 1.0"/>
+        </material>
+      </visual>
+      <collision>
+        <geometry>
+          <mesh filename="package://hexapod_description/meshes/micro-switch-tip.stl" scale="0.01 0.01 0.01"/>
+        </geometry>
+        <origin xyz="0 0 0" rpy="0 0 3.14"/>
+      </collision>
+      <inertial>
+        <mass value="0.01"/>
+        <origin xyz="0 0 0" rpy="0 0 0"/>
+        <inertia ixx="0.00001" ixy="0.0" ixz="0.0" iyy="0.00001" iyz="0.0" izz="0.00001"/>
+      </inertial>
+    </link>
+    <joint name="${prefix}_micro_switch_tip_joint" type="fixed">
+      <parent link="${prefix}_tibia_link"/>
+      <child link="${prefix}_micro_switch_tip_link"/>
+      <origin xyz="0.4 0 -1.3" rpy="0 0 0"/>
+    </joint>
+    <link name="${prefix}_tip_link">
+      <visual>
+        <geometry>
+          <mesh filename="package://hexapod_description/meshes/tip.stl" scale="0.01 0.01 0.01"/>
+        </geometry>
+        <origin xyz="0 0 0" rpy="0 0 0"/>
+        <material name="orange">
+          <color rgba="1.0 0.5 0.0 1.0"/>
+        </material>
+      </visual>
+      <collision>
+        <geometry>
+          <mesh filename="package://hexapod_description/meshes/tip.stl" scale="0.01 0.01 0.01"/>
+        </geometry>
+        <origin xyz="0 0 0" rpy="0 0 0"/>
+      </collision>
+      <inertial>
+        <mass value="0.01"/>
+        <origin xyz="0 0 0" rpy="0 0 0"/>
+        <inertia ixx="0.00001" ixy="0.0" ixz="0.0" iyy="0.00001" iyz="0.0" izz="0.00001"/>
+      </inertial>
+    </link>
+    <joint name="${prefix}_tip_joint" type="fixed">
+      <parent link="${prefix}_micro_switch_tip_link"/>
+      <child link="${prefix}_tip_link"/>
+      <origin xyz="0 0 0" rpy="0 0 0"/>
+    </joint>
   </xacro:macro>
 </robot>

File: hexapod_ws/src/hexapod_description/urdf/single_leg.urdf.xacro (robot description, xacro)
@@ -1,31 +1,10 @@
 <?xml version="1.0"?>
 <robot xmlns:xacro="http://www.ros.org/wiki/xacro" name="single_leg_test">
-  <material name="orange">
-    <color rgba="1.0 0.5 0.0 1.0"/>
-  </material>
-  <material name="grey">
-    <color rgba="0.5 0.5 0.5 1.0"/>
-  </material>
-  <link name="base_link">
-    <visual>
-      <geometry>
-        <box size="0.1 0.1 0.1"/>
-      </geometry>
-      <material name="grey"/>
-    </visual>
-    <collision>
-      <geometry>
-        <box size="0.1 0.1 0.1"/>
-      </geometry>
-    </collision>
-    <inertial>
-      <mass value="1.0"/>
-      <origin xyz="0 0 0" rpy="0 0 0"/>
-      <inertia ixx="0.01" ixy="0.0" ixz="0.0" iyy="0.01" iyz="0.0" izz="0.01"/>
-    </inertial>
-  </link>
-  <!-- Підключаємо файл макросу ноги -->
+  <!-- Тільки порожній базовий лінк -->
+  <link name="base_link"/>
+  <!-- Підключаємо макрос ноги -->
   <xacro:include filename="$(find hexapod_description)/urdf/leg.urdf.xacro"/>
-  <!-- Викликаємо макрос для однієї лівої ноги (side="left", префікс="left_front") -->
-  <xacro:hexapod_leg side="left" prefix="left_front" x_pos="0.0" y_pos="0.0" yaw_rot="0.0"/>
+  <!-- Викликаємо одну ногу -->
+  <xacro:hexapod_leg side="left" prefix="l1" x_pos="-0.6" y_pos="0.8" z_pos="0.0" yaw_rot="2.35"/>
+  <xacro:hexapod_leg side="right" prefix="r1" x_pos="0.6" y_pos="0.8" z_pos="0.0" yaw_rot="0.78"/>
 </robot>

Commit message: rm: physics in urdf

File: hexapod_ws/src/hexapod_description/urdf/leg.urdf.xacro (robot description, xacro)
@@ -19,7 +19,5 @@
       </collision>
       <inertial>
-        <mass value="0.05"/>
         <origin xyz="0 0 0" rpy="0 0 0"/>
-        <inertia ixx="0.0001" ixy="0.0" ixz="0.0" iyy="0.0001" iyz="0.0" izz="0.0001"/>
       </inertial>
     </link>
@@ -48,7 +46,5 @@
       </collision>
       <inertial>
-        <mass value="0.08"/>
         <origin xyz="0 0 0" rpy="0 0 0"/>
-        <inertia ixx="0.0001" ixy="0.0" ixz="0.0" iyy="0.0001" iyz="0.0" izz="0.0001"/>
       </inertial>
     </link>
@@ -77,7 +73,5 @@
       </collision>
       <inertial>
-        <mass value="0.05"/>
         <origin xyz="0 0 0" rpy="0 0 0"/>
-        <inertia ixx="0.0001" ixy="0.0" ixz="0.0" iyy="0.0001" iyz="0.0" izz="0.0001"/>
       </inertial>
     </link>
@@ -106,7 +100,5 @@
       </collision>
       <inertial>
-        <mass value="0.01"/>
         <origin xyz="0 0 0" rpy="0 0 0"/>
-        <inertia ixx="0.00001" ixy="0.0" ixz="0.0" iyy="0.00001" iyz="0.0" izz="0.00001"/>
       </inertial>
     </link>
@@ -133,7 +125,5 @@
       </collision>
       <inertial>
-        <mass value="0.01"/>
         <origin xyz="0 0 0" rpy="0 0 0"/>
-        <inertia ixx="0.00001" ixy="0.0" ixz="0.0" iyy="0.00001" iyz="0.0" izz="0.00001"/>
       </inertial>
     </link>
@@ -160,7 +150,5 @@
       </collision>
       <inertial>
-        <mass value="0.01"/>
         <origin xyz="0 0 0" rpy="0 0 0"/>
-        <inertia ixx="0.00001" ixy="0.0" ixz="0.0" iyy="0.00001" iyz="0.0" izz="0.00001"/>
       </inertial>
     </link>

Commit message: fix: automate launch

File: hexapod_ws/src/hexapod_description/urdf/leg.urdf.xacro (robot description, xacro)
@@ -32,5 +32,6 @@
       <origin xyz="${x_pos} ${y_pos} ${z_pos}" rpy="0 0 ${yaw_rot}"/>
       <axis xyz="0 0 1"/>
-      <limit lower="-1.57" upper="1.57" effort="2.0" velocity="1.0"/>
+      <limit lower="-1.57" upper="1.57" effort="100.0" velocity="3.0"/>
+      <dynamics damping="0.5" friction="0.05"/>
     </joint>
     <link name="${prefix}_femur_link">
@@ -64,5 +65,6 @@
       <origin xyz="0.4 0 0.05" rpy="0 -0.78 0"/>
       <axis xyz="0 1 0"/>
-      <limit lower="-1.57" upper="1.57" effort="2.0" velocity="1.0"/>
+      <limit lower="-1.57" upper="1.57" effort="100.0" velocity="3.0"/>
+      <dynamics damping="0.5" friction="0.05"/>
     </joint>
     <link name="${prefix}_tibia_link">
@@ -96,5 +98,6 @@
       <origin xyz="0.8 0 0" rpy="0 0.78 0"/>
       <axis xyz="0 1 0"/>
-      <limit lower="-1.57" upper="1.57" effort="2.0" velocity="1.0"/>
+      <limit lower="-1.57" upper="1.57" effort="100.0" velocity="3.0"/>
+      <dynamics damping="0.5" friction="0.05"/>
     </joint>
     <link name="${prefix}_shield_link">

Commit message: fix: tibia link y coordinate

File: hexapod_ws/src/hexapod_description/urdf/leg.urdf.xacro (robot description, xacro)
@@ -59,5 +59,5 @@
                 scale="0.001 0.001 0.001"/>
         </geometry>
-        <origin xyz="0.05 -0.005 0" rpy="0 0 3.14"/>
+        <origin xyz="0.05 ${-0.005 if side == 'left' else 0.005} 0" rpy="0 0 3.14"/>
         <material name="orange">
           <color rgba="1.0 0.5 0.0 1.0"/>
